Commit message: Adicionando nav2 ao platform, sem os sensores, mas esta com paramentros e mapa

File: robotics_ws/src/rav_description/urdf/platform_with_mesh_and_wheels.urdf.xacro (robot description, xacro)
@@ -10,6 +10,6 @@
   <xacro:property name="platform_mesh_scale" value="0.001 0.001 0.001"/>
   <!-- Rodas (mantendo a ideia da sua URDF antiga) -->
-  <xacro:property name="wheel_radius" value="0.08"/>
-  <xacro:property name="wheel_width"  value="0.05"/>
+  <xacro:property name="wheel_radius" value="0.07"/>
+  <xacro:property name="wheel_width"  value="0.038"/>
   <!-- Mantendo o seu wheel_y / wheel_z (do jeito que você configurou antes) -->
   <xacro:property name="platform_diameter" value="0.50"/>
@@ -27,5 +27,5 @@
     <visual>
       <!-- Se o STL já estiver orientado certinho, deixa 0 0 0 -->
-      <origin xyz="-0.86 -0.25 0.04" rpy="0 0 0"/>
+      <origin xyz="0 0 0.048" rpy="0 0 1.57"/>
       <geometry>
         <mesh filename="package://rav_description/meshes/${platform_mesh}" scale="${platform_mesh_scale}"/>
@@ -33,5 +33,5 @@
     </visual>
     <collision>
-      <origin xyz="-0.86 -0.25 0.04" rpy="0 0 0"/>
+      <origin xyz="-0.86 -0.25 0.04" rpy="0 0 1.57"/>
       <geometry>
         <mesh filename="package://rav_description/meshes/${platform_mesh}" scale="${platform_mesh_scale}"/>

Commit message: juncao da urdf corpo e platform navegando no rviz

File: robotics_ws/src/rav_description/urdf/platform_with_mesh_and_wheels.urdf.xacro (robot description, xacro)
@@ -1,97 +1,72 @@
 <?xml version="1.0"?>
 <robot name="rav_platform" xmlns:xacro="http://www.ros.org/wiki/xacro">
-  <!-- ===================== -->
-  <!--   PARÂMETROS GERAIS   -->
-  <!-- ===================== -->
-  <!-- Troque pelo nome do seu STL dentro de rav_description/meshes -->
-  <xacro:property name="platform_mesh" value="platform.dae"/>
-  <!-- Se o STL estiver em milímetros (muito comum), use scale="0.001 0.001 0.001"
-       Se estiver em metros, use 1 1 1 -->
-  <xacro:property name="platform_mesh_scale" value="0.001 0.001 0.001"/>
-  <!-- Rodas (mantendo a ideia da sua URDF antiga) -->
-  <xacro:property name="wheel_radius" value="0.07"/>
-  <xacro:property name="wheel_width"  value="0.038"/>
-  <!-- Mantendo o seu wheel_y / wheel_z (do jeito que você configurou antes) -->
-  <xacro:property name="platform_diameter" value="0.50"/>
-  <xacro:property name="platform_radius" value="${platform_diameter/2.0}"/>
-  <!-- Atenção: você tinha esse offset -0.43; estou mantendo porque você pediu
-       para considerar suas origens. Se ficar esquisito, a gente ajusta depois. -->
-  <xacro:property name="wheel_y" value="${platform_radius + wheel_width/2.0 - 0.43}"/>
-  <xacro:property name="wheel_z" value="${wheel_radius}"/>
-  <!-- ===================== -->
-  <!--        LINKS          -->
-  <!-- ===================== -->
-  <link name="base_link"/>
-  <!-- Base do Platform usando STL -->
-  <link name="platform_base_link">
-    <visual>
-      <!-- Se o STL já estiver orientado certinho, deixa 0 0 0 -->
-      <origin xyz="0 0 0.048" rpy="0 0 1.57"/>
-      <geometry>
-        <mesh filename="package://rav_description/meshes/${platform_mesh}" scale="${platform_mesh_scale}"/>
-      </geometry>
-    </visual>
-    <collision>
-      <origin xyz="-0.86 -0.25 0.04" rpy="0 0 1.57"/>
-      <geometry>
-        <mesh filename="package://rav_description/meshes/${platform_mesh}" scale="${platform_mesh_scale}"/>
-      </geometry>
-    </collision>
-    <!-- Inércia placeholder (ok para RViz) -->
-    <inertial>
-      <origin xyz="-0.86 -0.25 0.04" rpy="0 0 0"/>
-      <mass value="35.0"/>
-      <inertia ixx="1.0" ixy="0.0" ixz="0.0" iyy="1.0" iyz="0.0" izz="1.0"/>
-    </inertial>
-  </link>
-  <joint name="base_to_platform" type="fixed">
-    <parent link="base_link"/>
-    <child link="platform_base_link"/>
-    <origin xyz="0 0 0" rpy="0 0 0"/>
-  </joint>
-  <!-- ===================== -->
-  <!--         RODAS         -->
-  <!-- ===================== -->
-  <!-- Roda esquerda -->
-  <link name="wheel_left_link">
-    <visual>
-      <origin xyz="0 0 0" rpy="1.57 0 0"/>
-      <geometry>
-        <cylinder radius="${wheel_radius}" length="${wheel_width}"/>
-      </geometry>
-      <material name="wheel_black">
-        <color rgba="0.05 0.05 0.05 1.0"/>
-      </material>
-    </visual>
-  </link>
-  <!-- ATENÇÃO:
-       - Se você quiser roda "animável" pelo joint_state_publisher, use continuous.
-       - Se você só quer visual, use fixed.
-       Vou deixar continuous porque você já estava nessa direção. -->
-  <joint name="wheel_left_joint" type="continuous">
-    <parent link="platform_base_link"/>
-    <child link="wheel_left_link"/>
-    <!-- Mantendo sua origem via wheel_y / wheel_z -->
-    <origin xyz="0 ${wheel_y} ${wheel_z}" rpy="0 0 0"/>
-    <!-- Eixo mantido como você usou -->
-    <axis xyz="0 1 0"/>
-  </joint>
-  <!-- Roda direita -->
-  <link name="wheel_right_link">
-    <visual>
-      <origin xyz="0 0 0" rpy="1.57 0 0"/>
-      <geometry>
-        <cylinder radius="${wheel_radius}" length="${wheel_width}"/>
-      </geometry>
-      <material name="wheel_black">
-        <color rgba="0.05 0.05 0.05 1.0"/>
-      </material>
-    </visual>
-  </link>
-  <joint name="wheel_right_joint" type="continuous">
-    <parent link="platform_base_link"/>
-    <child link="wheel_right_link"/>
-    <origin xyz="0 ${-wheel_y} ${wheel_z}" rpy="0 0 0"/>
-    <axis xyz="0 1 0"/>
-  </joint>
+  <xacro:macro name="rav_platform" params="">
+    <xacro:property name="platform_mesh" value="platform.dae"/>
+    <xacro:property name="platform_mesh_scale" value="0.001 0.001 0.001"/>
+    <xacro:property name="wheel_radius" value="0.07"/>
+    <xacro:property name="wheel_width"  value="0.038"/>
+    <xacro:property name="platform_diameter" value="0.50"/>
+    <xacro:property name="platform_radius" value="${platform_diameter/2.0}"/>
+    <xacro:property name="wheel_y" value="${platform_radius + wheel_width/2.0 - 0.43}"/>
+    <xacro:property name="wheel_z" value="${wheel_radius}"/>
+    <link name="base_link"/>
+    <link name="platform_base_link">
+      <visual>
+        <origin xyz="0 0 0.048" rpy="0 0 1.57"/>
+        <geometry>
+          <mesh filename="package://rav_description/meshes/${platform_mesh}" scale="${platform_mesh_scale}"/>
+        </geometry>
+      </visual>
+      <collision>
+        <origin xyz="-0.86 -0.25 0.04" rpy="0 0 1.57"/>
+        <geometry>
+          <mesh filename="package://rav_description/meshes/${platform_mesh}" scale="${platform_mesh_scale}"/>
+        </geometry>
+      </collision>
+      <inertial>
+        <origin xyz="-0.86 -0.25 0.04" rpy="0 0 0"/>
+        <mass value="35.0"/>
+        <inertia ixx="1.0" ixy="0.0" ixz="0.0" iyy="1.0" iyz="0.0" izz="1.0"/>
+      </inertial>
+    </link>
+    <joint name="base_to_platform" type="fixed">
+      <parent link="base_link"/>
+      <child link="platform_base_link"/>
+      <origin xyz="0 0 0" rpy="0 0 0"/>
+    </joint>
+    <link name="wheel_left_link">
+      <visual>
+        <origin xyz="0 0 0" rpy="1.57 0 0"/>
+        <geometry>
+          <cylinder radius="${wheel_radius}" length="${wheel_width}"/>
+        </geometry>
+        <material name="wheel_black">
+          <color rgba="0.05 0.05 0.05 1.0"/>
+        </material>
+      </visual>
+    </link>
+    <joint name="wheel_left_joint" type="continuous">
+      <parent link="platform_base_link"/>
+      <child link="wheel_left_link"/>
+      <origin xyz="0 ${wheel_y} ${wheel_z}" rpy="0 0 0"/>
+      <axis xyz="0 1 0"/>
+    </joint>
+    <link name="wheel_right_link">
+      <visual>
+        <origin xyz="0 0 0" rpy="1.57 0 0"/>
+        <geometry>
+          <cylinder radius="${wheel_radius}" length="${wheel_width}"/>
+        </geometry>
+        <material name="wheel_black">
+          <color rgba="0.05 0.05 0.05 1.0"/>
+        </material>
+      </visual>
+    </link>
+    <joint name="wheel_right_joint" type="continuous">
+      <parent link="platform_base_link"/>
+      <child link="wheel_right_link"/>
+      <origin xyz="0 ${-wheel_y} ${wheel_z}" rpy="0 0 0"/>
+      <axis xyz="0 1 0"/>
+    </joint>
+  </xacro:macro>
 </robot>

File: robotics_ws/src/rav_description/urdf/rav_body.urdf (robot description, URDF)
Before this commit: robot rav_body, 2 links, 1 joints
Links:
- link body_link: geometry collision mesh filename=../meshes/RAV_BODY.dae scale=0.001 0.001 0.001; visual mesh filename=../meshes/RAV_BODY.dae scale=0.001 0.001 0.001
