Commit message: adicionando manip na urdf geral mas falta arrumar joint state publisher

File: robotics_ws/src/rav_description/urdf/arm.urdf.xacro (robot description, xacro)
@@ -68,47 +68,7 @@
       <xacro:inertial_block mass="${0.001}" length="${0.001}" radius="${0.001}"/>
     </link>
-    <joint name="${prefix}joint_1_fixed" type="fixed">
+    <joint name="${prefix}joint_2" type="revolute">
       <origin xyz="0 0 0" rpy="0 0 0"/>
       <parent link="${prefix}base_link"/>
-      <child link="${prefix}link_1"/>
-    </joint>
-    <link name="${prefix}link_1">
-      <xacro:inertial_block mass="${mass_2}" length="${length_2}" radius="${radius_2}"/>
-      <visual>
-        <origin xyz="0 0 ${length_2/2.0}" rpy="0 0 0"/>
-        <geometry><cylinder radius="${radius_2}" length="${length_2}"/></geometry>
-        <material name="Grey"/>
-      </visual>
-      <collision>
-        <origin xyz="0 0 ${length_2/2.0}" rpy="0 0 0"/>
-        <geometry><cylinder radius="${radius_2}" length="${length_2}"/></geometry>
-      </collision>
-    </link>
-    <xacro:gazebo_grey_link_color_block link_name="${prefix}link_1"/>
-    <link name="${prefix}link_1_endlink">
-      <xacro:inertial_block mass="${mass_2/3.0}" length="${2*radius_2+2*radius_3}" radius="${radius_2}"/>
-      <visual>
-        <origin xyz="0 0 ${(2*radius_2+2*radius_3)/2.0}" rpy="0 0 0"/>
-        <geometry><cylinder radius="${radius_2*1.1}" length="${2*radius_2+2*radius_3}"/></geometry>
-        <material name="LightBlue"/>
-      </visual>
-      <collision>
-        <origin xyz="0 0 ${(2*radius_2+2*radius_3)/2.0}" rpy="0 0 0"/>
-        <geometry><cylinder radius="${radius_2*1.1}" length="${2*radius_2+2*radius_3}"/></geometry>
-      </collision>
-    </link>
-    <xacro:gazebo_blue_link_color_block link_name="${prefix}link_1_endlink"/>
-    <joint name="${prefix}link_1_endjoint" type="fixed">
-      <origin xyz="${-radius_2} 0 ${length_2 - 0.01}" rpy="0 ${M_PI/2.0} 0"/>
-      <parent link="${prefix}link_1"/>
-      <child link="${prefix}link_1_endlink"/>
-    </joint>
-    <gazebo reference="${prefix}link_1_endjoint">
-      <disableFixedJointLumping>true</disableFixedJointLumping>
-      <preserveFixedJoint>true</preserveFixedJoint>
-    </gazebo>
-    <joint name="${prefix}joint_2" type="revolute">
-      <origin xyz="${radius_2 + radius_3} 0 ${length_2}" rpy="0 0 0"/>
-      <parent link="${prefix}link_1"/>
       <child link="${prefix}link_2"/>
       <axis xyz="1 0 0"/>

File: robotics_ws/src/rav_description/urdf/rav_complete.urdf.xacro (robot description, xacro)
@@ -3,12 +3,12 @@
   <xacro:include filename="$(find rav_description)/urdf/platform_with_mesh_and_wheels.urdf.xacro"/>
   <xacro:include filename="$(find rav_description)/urdf/rav_body.urdf.xacro"/>
-  <!-- <xacro:include filename="$(find rav_description)/urdf/arm.urdf.xacro"/> -->
+  <xacro:include filename="$(find rav_description)/urdf/arm.urdf.xacro"/>
   <xacro:rav_platform/>
   <xacro:rav_body parent_link="platform_base_link" xyz="0 0 0.2572" rpy="0 0 0"/>
   <!-- Braço montado sobre o corpo do robô -->
-  <!-- <xacro:arm
+  <xacro:arm
     parent_link="platform_base_link"
     prefix="arm_"
-    xyz="0 0 0.2572"
-    rpy="0 0 0"/> -->
+    xyz="0 1 0.69"
+    rpy="0 0 1.57"/>
 </robot>

Commit message: urdf manip junto com outras urdf e motores do manip funionando. (use_gui:=true para ligar joint state publisher)

File: robotics_ws/src/rav_description/urdf/arm.urdf.xacro (robot description, xacro)
@@ -1,4 +1,5 @@
 <?xml version="1.0"?>
 <robot xmlns:xacro="http://www.ros.org/wiki/xacro" name="arm">
+  <xacro:arg name="use_sim" default="false"/>
   <xacro:macro name="arm" params="parent_link prefix xyz:='0 0 0' rpy:='0 0 0'">
     <xacro:property name="M_PI" value="3.14159"/>
@@ -207,39 +208,41 @@
       </collision>
     </link>
-    <ros2_control name="${prefix}GazeboSystem" type="system">
-      <hardware>
-        <plugin>gazebo_ros2_control/GazeboSystem</plugin>
-      </hardware>
-      <joint name="${prefix}joint_2">
-        <command_interface name="position"/>
-        <state_interface name="position"/>
-        <state_interface name="velocity"/>
-      </joint>
-      <joint name="${prefix}joint_3">
-        <command_interface name="position"/>
-        <state_interface name="position"/>
-        <state_interface name="velocity"/>
-      </joint>
-      <joint name="${prefix}joint_4">
-        <command_interface name="position"/>
-        <state_interface name="position"/>
-        <state_interface name="velocity"/>
-      </joint>
-      <joint name="${prefix}gripper_joint_1">
-        <command_interface name="position"/>
-        <state_interface name="position"/>
-        <state_interface name="velocity"/>
-      </joint>
-      <joint name="${prefix}gripper_joint_2">
-        <command_interface name="position"/>
-        <state_interface name="position"/>
-        <state_interface name="velocity"/>
-      </joint>
-    </ros2_control>
-    <gazebo>
-      <plugin filename="libgazebo_ros2_control.so" name="${prefix}gazebo_ros2_control">
-        <parameters>$(find rav_description)/config/arm_controllers.yaml</parameters>
-      </plugin>
-    </gazebo>
+    <xacro:if value="$(arg use_sim)">
+      <ros2_control name="${prefix}GazeboSystem" type="system">
+        <hardware>
+          <plugin>gazebo_ros2_control/GazeboSystem</plugin>
+        </hardware>
+        <joint name="${prefix}joint_2">
+          <command_interface name="position"/>
+          <state_interface name="position"/>
+          <state_interface name="velocity"/>
+        </joint>
+        <joint name="${prefix}joint_3">
+          <command_interface name="position"/>
+          <state_interface name="position"/>
+          <state_interface name="velocity"/>
+        </joint>
+        <joint name="${prefix}joint_4">
+          <command_interface name="position"/>
+          <state_interface name="position"/>
+          <state_interface name="velocity"/>
+        </joint>
+        <joint name="${prefix}gripper_joint_1">
+          <command_interface name="position"/>
+          <state_interface name="position"/>
+          <state_interface name="velocity"/>
+        </joint>
+        <joint name="${prefix}gripper_joint_2">
+          <command_interface name="position"/>
+          <state_interface name="position"/>
+          <state_interface name="velocity"/>
+        </joint>
+      </ros2_control>
+      <gazebo>
+        <plugin filename="libgazebo_ros2_control.so" name="${prefix}gazebo_ros2_control">
+          <parameters>$(find rav_description)/config/arm_controllers.yaml</parameters>
+        </plugin>
+      </gazebo>
+    </xacro:if>
   </xacro:macro>
 </robot>

Commit message: alteração na urdf do manip

File: robotics_ws/src/rav_description/urdf/arm.urdf.xacro (robot description, xacro)
@@ -12,14 +12,21 @@
     <xacro:property name="radius_1" value="0.1"/>
     <xacro:property name="radius_2" value="0.05"/>
-    <xacro:property name="radius_3" value="0.035"/>
+    <xacro:property name="radius_3" value="0.025"/>
     <xacro:property name="radius_4" value="0.025"/>
-    <xacro:property name="radius_5" value="0.025"/>
+    <xacro:property name="radius_5" value="0.022"/>
     <xacro:property name="radius_6" value="0.02"/>
     <xacro:property name="length_1" value="0.15"/>
+    <xacro:property name="length_2" value="0.4"/>
+    <xacro:property name="length_3" value="0.4"/>
+    <xacro:property name="length_4" value="0.2"/>
+    <xacro:property name="length_5" value="0.12"/>
+    <xacro:property name="length_6" value="0.07"/>
+    <!-- Original -->
+    <!-- <xacro:property name="length_1" value="0.15"/>
     <xacro:property name="length_2" value="0.4"/>
     <xacro:property name="length_3" value="0.5"/>
     <xacro:property name="length_4" value="0.3"/>
     <xacro:property name="length_5" value="0.15"/>
-    <xacro:property name="length_6" value="0.07"/>
+    <xacro:property name="length_6" value="0.07"/> -->
     <material name="Black"><color rgba="0.0 0.0 0.0 1.0"/></material>
     <material name="Red"><color rgba="0.8 0.0 0.0 1.0"/></material>
@@ -67,8 +74,21 @@
     </joint>
     <link name="${prefix}base_link">
-      <xacro:inertial_block mass="${0.001}" length="${0.001}" radius="${0.001}"/>
+      <xacro:inertial_block mass="${mass_3/4.0}" length="${radius_3*2.0}" radius="${radius_3*1.6}"/>
+      <visual>
+      <origin xyz="0 0 ${radius_3*1.6}" rpy="0 ${M_PI/2.0} 0"/>
+      <geometry>
+        <cylinder radius="${radius_3*1.6}" length="${radius_3*2.0}"/>
+      </geometry>
+      <material name="LightBlue"/>
+    </visual>
+    <collision>
+      <origin xyz="0 0 ${radius_3*1.6}" rpy="0 ${M_PI/2.0} 0"/>
+      <geometry>
+        <cylinder radius="${radius_3*1.6}" length="${radius_3*2.0}"/>
+      </geometry>
+    </collision>
     </link>
     <joint name="${prefix}joint_2" type="revolute">
-      <origin xyz="0 0 0" rpy="0 0 0"/>
+      <origin xyz="0 0 ${radius_3*1.6}" rpy="0 0 0"/>
       <parent link="${prefix}base_link"/>
       <child link="${prefix}link_2"/>
@@ -90,16 +110,19 @@
     <xacro:gazebo_grey_link_color_block link_name="${prefix}link_2"/>
     <link name="${prefix}link_2_endlink">
-      <xacro:inertial_block mass="${mass_3/3.0}" length="${2*radius_3+2*radius_4}" radius="${radius_3}"/>
-      <visual>
-        <origin xyz="0 0 ${(2*radius_3+2*radius_4)/2.0}" rpy="0 0 0"/>
-        <geometry><cylinder radius="${radius_3*1.1}" length="${2*radius_3+2*radius_4}"/></geometry>
+      <xacro:inertial_block mass="${mass_3/4.0}" length="${radius_3*2.0}" radius="${radius_3}"/>
+      <visual>
+        <origin xyz="0 0 ${radius_3}" rpy="0 0 0"/>
+        <geometry>
+          <cylinder radius="${radius_3*2}" length="${radius_3*2.0}"/>
+        </geometry>
         <material name="LightBlue"/>
       </visual>
       <collision>
-        <origin xyz="0 0 ${(2*radius_3+2*radius_4)/2.0}" rpy="0 0 0"/>
-        <geometry><cylinder radius="${radius_3*1.1}" length="${2*radius_3+2*radius_4}"/></geometry>
-      </collision>
-    </link>
-    <xacro:gazebo_blue_link_color_block link_name="${prefix}link_2_endlink"/>
+        <origin xyz="0 0 ${radius_3}" rpy="0 0 0"/>
+        <geometry>
+          <cylinder radius="${radius_3*2}" length="${radius_3*2.0}"/>
+        </geometry>
+      </collision>
+    </link>
     <joint name="${prefix}link_2_endjoint" type="fixed">
       <origin xyz="${-radius_3} 0 ${length_3 - 0.01}" rpy="0 ${M_PI/2.0} 0"/>
@@ -112,5 +135,5 @@
     </gazebo>
     <joint name="${prefix}joint_3" type="revolute">
-      <origin xyz="${radius_3 + radius_4} 0 ${length_3 - radius_3}" rpy="0 0 0"/>
+      <origin xyz="0 0 ${length_3}" rpy="0 0 0"/>
       <parent link="${prefix}link_2"/>
       <child link="${prefix}link_3"/>
@@ -120,13 +143,17 @@
     <link name="${prefix}link_3">
       <xacro:inertial_block mass="${mass_4}" length="${length_4}" radius="${radius_4}"/>
-      <visual>
-        <origin xyz="0 0 ${length_4/2.0}" rpy="0 0 0"/>
-        <geometry><cylinder radius="${radius_4}" length="${length_4}"/></geometry>
-        <material name="Grey"/>
-      </visual>
-      <collision>
-        <origin xyz="0 0 ${length_4/2.0}" rpy="0 0 0"/>
-        <geometry><cylinder radius="${radius_4}" length="${length_4}"/></geometry>
-      </collision>
+          <visual>
+      <origin xyz="0 0 ${(length_4 - radius_5*1.3)/2.0}" rpy="0 0 0"/>
+      <geometry>
+        <cylinder radius="${radius_4}" length="${length_4 - radius_5*1.3}"/>
+      </geometry>
+      <material name="Grey"/>
+    </visual>
+    <collision>
+      <origin xyz="0 0 ${(length_4 - radius_5*1.3)/2.0}" rpy="0 0 0"/>
+      <geometry>
+        <cylinder radius="${radius_4}" length="${length_4 - radius_5*1.3}"/>
+      </geometry>
+    </collision>
     </link>
     <xacro:gazebo_grey_link_color_block link_name="${prefix}link_3"/>
@@ -140,31 +167,49 @@
     <link name="${prefix}link_4">
       <xacro:inertial_block mass="${mass_5}" length="${length_5}" radius="${radius_5}"/>
-      <visual>
-        <origin xyz="0 0 ${radius_5/2.0}" rpy="0 ${M_PI/2.0} 0"/>
-        <geometry><box size="${radius_5*2} ${radius_5*2} ${length_5}"/></geometry>
-        <material name="Grey"/>
-      </visual>
-      <collision>
-        <origin xyz="0 0 ${radius_5/2.0}" rpy="0 0 0"/>
-        <geometry><box size="${radius_5*2} ${radius_5*2} ${length_5}"/></geometry>
-      </collision>
-    </link>
-    <xacro:gazebo_grey_link_color_block link_name="${prefix}link_4"/>
+      <!-- Cilindro da junta 4 -->
+      <visual>
+        <origin xyz="0 0 0" rpy="0 ${M_PI/2.0} 0"/>
+        <geometry>
+          <cylinder radius="${radius_5*1.3}" length="${radius_5*2.0}"/>
+        </geometry>
+        <material name="LightBlue"/>
+      </visual>
+      <collision>
+        <origin xyz="0 0 0" rpy="0 ${M_PI/2.0} 0"/>
+        <geometry>
+          <cylinder radius="${radius_5*1.3}" length="${radius_5*2.0}"/>
+        </geometry>
+      </collision>
+      <!-- Retângulo apoiado no limite superior do cilindro -->
+      <visual>
+        <origin xyz="0 0 ${radius_5*2.3}" rpy="0 ${M_PI/2.0} 0"/>
+        <geometry>
+          <box size="${radius_5*2} ${radius_5*2} ${length_5}"/>
+        </geometry>
+        <material name="Grey"/>
+      </visual>
+      <collision>
+        <origin xyz="0 0 ${radius_5*2.3}" rpy="0 ${M_PI/2.0} 0"/>
+        <geometry>
+          <box size="${radius_5*2} ${radius_5*2} ${length_5}"/>
+        </geometry>
+      </collision>
+    </link>
     <joint name="${prefix}gripper_joint_1" type="prismatic">
-      <origin xyz="0 0 ${radius_5 + length_6/2.0}" rpy="0 0 0"/>
+      <origin xyz="0 0 ${radius_5*2.3 + length_6/2.0}" rpy="0 0 0"/>
       <parent link="${prefix}link_4"/>
       <child link="${prefix}gripper_link_1"/>
       <axis xyz="1 0 0"/>
-      <limit lower="${radius_6/2.0}" upper="0.05" effort="100.0" velocity="1.0"/>
+      <limit lower="${radius_6/2.0}" upper="0.03" effort="100.0" velocity="1.0"/>
     </joint>
     <joint name="${prefix}gripper_joint_2" type="prismatic">
-      <origin xyz="0 0 ${radius_5 + length_6/2.0}" rpy="0 0 0"/>
+      <origin xyz="0 0 ${radius_5*2.3 + length_6/2.0}" rpy="0 0 0"/>
       <parent link="${prefix}link_4"/>
       <child link="${prefix}gripper_link_2"/>
       <axis xyz="1 0 0"/>
-      <limit lower="-0.05" upper="${-radius_6/2.0}" effort="100.0" velocity="1.0"/>
+      <limit lower="-0.03" upper="${-radius_6/2.0}" effort="100.0" velocity="1.0"/>
     </joint>
     <joint name="${prefix}gripper_frame_joint" type="fixed">
-      <origin xyz="0 0 ${radius_5*2 + length_6/2 + 0.01}" rpy="0 0 0"/>
+      <origin xyz="0 0 ${radius_5*2.3 + length_6}" rpy="0 0 0"/>
       <parent link="${prefix}link_4"/>
       <child link="${prefix}gripper_frame_cp"/>

File: robotics_ws/src/rav_description/urdf/rav_complete.urdf.xacro (robot description, xacro)
@@ -10,5 +10,5 @@
     parent_link="platform_base_link"
     prefix="arm_"
-    xyz="0 1 0.69"
+    xyz="0.07 0 0.69"
     rpy="0 0 1.57"/>
 </robot>

Commit message: Arrumando a gripper

File: robotics_ws/src/rav_description/urdf/arm.urdf.xacro (robot description, xacro)
@@ -201,5 +201,5 @@
       <child link="${prefix}gripper_link_1"/>
       <axis xyz="1 0 0"/>
-      <limit lower="${radius_6/2.0}" upper="0.03" effort="100.0" velocity="1.0"/>
+      <limit lower="0.0" upper="0.03" effort="100.0" velocity="1.0"/>
     </joint>
     <joint name="${prefix}gripper_joint_2" type="prismatic">
@@ -207,6 +207,7 @@
       <parent link="${prefix}link_4"/>
       <child link="${prefix}gripper_link_2"/>
-      <axis xyz="1 0 0"/>
-      <limit lower="-0.03" upper="${-radius_6/2.0}" effort="100.0" velocity="1.0"/>
+      <axis xyz="-1 0 0"/>
+      <limit lower="0.0" upper="0.03" effort="100.0" velocity="1.0"/>
+      <mimic joint="${prefix}gripper_joint_1" multiplier="1.0" offset="0.0"/>
     </joint>
     <joint name="${prefix}gripper_frame_joint" type="fixed">

Commit message: pacote moveit

File: robotics_ws/src/rav_description/urdf/arm.urdf.xacro (robot description, xacro)
@@ -93,5 +93,5 @@
       <parent link="${prefix}base_link"/>
       <child link="${prefix}link_2"/>
-      <axis xyz="1 0 0"/>
+      <axis xyz="-1 0 0"/>
       <limit lower="0.0" upper="${M_PI * 2}" effort="300.0" velocity="1.0"/>
     </joint>
