Commit message: Integra manipulador, Gazebo, MoveIt e visao 3D

File: robotics_ws/src/rav_description/urdf/rav_manipulator.urdf.xacro (robot description, xacro)
@@ -15,4 +15,21 @@
 -->
 <robot name="rav_manipulator" xmlns:xacro="http://www.ros.org/wiki/xacro">
+  <!--
+    Propriedades físicas provisórias para Gazebo.
+    Não interferem no controle dos Dynamixel reais.
+    Substituir futuramente por massas e tensores medidos/calculados.
+  -->
+  <xacro:macro
+      name="rav_provisional_inertial"
+      params="mass xyz ixx iyy izz">
+    <inertial>
+      <origin xyz="${xyz}" rpy="0 0 0"/>
+      <mass value="${mass}"/>
+      <inertia
+          ixx="${ixx}" ixy="0.0" ixz="0.0"
+          iyy="${iyy}" iyz="0.0"
+          izz="${izz}"/>
+    </inertial>
+  </xacro:macro>
   <xacro:macro name="rav_manipulator"
                params="parent_link mount_xyz:='0 0 0' mount_rpy:='0 0 0' use_fake_hardware:=false">
@@ -56,4 +73,8 @@
     -->
     <link name="manipulator_base_link">
+      <xacro:rav_provisional_inertial
+          mass="1.0"
+          xyz="0 0 0"
+          ixx="0.004" iyy="0.004" izz="0.004"/>
       <visual>
         <origin xyz="0 0.047471563258 -0.733684638388" rpy="0 0 0"/>
@@ -86,4 +107,8 @@
     -->
     <link name="shoulder_link">
+      <xacro:rav_provisional_inertial
+          mass="1.5"
+          xyz="0 0.000015 0.139059"
+          ixx="0.010" iyy="0.010" izz="0.002"/>
       <visual>
         <origin xyz="0 0.047471563258 -0.733684638388" rpy="0 0 0"/>
@@ -132,4 +157,8 @@
     -->
     <link name="elbow_link">
+      <xacro:rav_provisional_inertial
+          mass="1.2"
+          xyz="0 -0.171515 0"
+          ixx="0.012" iyy="0.002" izz="0.012"/>
       <visual>
         <origin xyz="0 0.047441923275 -1.011802711307" rpy="0 0 0"/>
@@ -180,4 +209,8 @@
     <!-- U aço 3, onde o Dynamixel 4 será fixado quando a garra entrar. -->
     <link name="wrist_link">
+      <xacro:rav_provisional_inertial
+          mass="0.8"
+          xyz="0 0 0"
+          ixx="0.004" iyy="0.004" izz="0.004"/>
       <visual>
         <origin xyz="0 0.390472110866 -1.011787152338" rpy="0 0 0"/>
@@ -223,4 +256,24 @@
       </collision>
     </link>
+    <!--
+      Ponto terminal provisório do terceiro elo.
+      Não representa uma garra; representa a ponta física usada nos testes
+      de alcance do manipulador sem gripper.
+    -->
+    <link name="wrist_tip">
+      <visual>
+        <geometry>
+          <sphere radius="0.015"/>
+        </geometry>
+        <material name="wrist_tip_material">
+          <color rgba="1.0 0.0 0.0 1.0"/>
+        </material>
+      </visual>
+    </link>
+    <joint name="wrist_tip_joint" type="fixed">
+      <parent link="wrist_link"/>
+      <child link="wrist_tip"/>
+      <origin xyz="0 -0.120 0" rpy="0 0 0"/>
+    </joint>
     <!-- Frame neutro para a futura garra. A posição final ainda não foi presumida. -->
     <link name="gripper_mount"/>

File: robotics_ws/src/rav_manipulator_moveit_config/config/rav_manipulator_dynamixel_real_unmounted.urdf.xacro (robot description, xacro)
@@ -18,6 +18,6 @@
       <param name="device">/dev/serial/by-id/usb-CM-900_ROBOTIS_Virtual_COM_Port-if00</param>
       <param name="baud">1000000</param>
-      <param name="profile_velocity">25</param>
-      <param name="profile_acceleration">8</param>
+      <param name="profile_velocity">35</param>
+      <param name="profile_acceleration">12</param>
     </hardware>
     <joint name="shoulder_joint">

Commit message: Atualiza geometria dos links 1 e 2 do manipulador

File: robotics_ws/src/rav_description/urdf/rav_manipulator.urdf.xacro (robot description, xacro)
@@ -44,6 +44,6 @@
     -->
     <xacro:property name="j1_to_j2_y" value="0.000029639983"/>
-    <xacro:property name="j1_to_j2_z" value="0.278118072919"/>
-    <xacro:property name="j2_to_j3_y" value="-0.343030187591"/>
+    <xacro:property name="j1_to_j2_z" value="0.289118072919"/>
+    <xacro:property name="j2_to_j3_y" value="-0.334030187591"/>
     <xacro:property name="j2_to_j3_z" value="-0.000015558969"/>
     <!-- Limites provisórios: somente para RViz/MoveIt sem hardware real. -->
@@ -128,5 +128,5 @@
       <!-- Corpo do Dynamixel 2, fixo no Link 1. -->
       <visual>
-        <origin xyz="0 0.047501203241 -0.455566565469" rpy="0 0 0"/>
+        <origin xyz="0 0.047501203241 -0.444566565469" rpy="0 0 0"/>
         <geometry>
           <mesh filename="package://rav_description/meshes/manipulator/dynamixel_xm540.stl"
@@ -136,5 +136,5 @@
       </visual>
       <collision>
-        <origin xyz="0 0.047501203241 -0.455566565469" rpy="0 0 0"/>
+        <origin xyz="0 0.047501203241 -0.444566565469" rpy="0 0 0"/>
         <geometry>
           <mesh filename="package://rav_description/meshes/manipulator/dynamixel_xm540.stl"
@@ -183,5 +183,5 @@
       -->
       <visual>
-        <origin xyz="0 0.390654450797 0.047456004289" rpy="1.57079632679 0 0"/>
+        <origin xyz="0 0.399654450797 0.047456004289" rpy="1.57079632679 0 0"/>
         <geometry>
           <mesh filename="package://rav_description/meshes/manipulator/dynamixel_xm540.stl"
@@ -191,5 +191,5 @@
       </visual>
       <collision>
-        <origin xyz="0 0.390654450797 0.047456004289" rpy="1.57079632679 0 0"/>
+        <origin xyz="0 0.399654450797 0.047456004289" rpy="1.57079632679 0 0"/>
         <geometry>
           <mesh filename="package://rav_description/meshes/manipulator/dynamixel_xm540.stl"
