Commit message: ädicionando urdf gripper

File: robotics_ws/src/rav_description/urdf/rav_manipulator.urdf.xacro (robot description, xacro)
@@ -1,23 +1,19 @@
 <?xml version="1.0"?>
 <!--
-  Modelo do manipulador do TCC do RAV.
-  Escopo desta primeira etapa
-  - 3 juntas revolutas: shoulder_joint, elbow_joint e wrist_joint.
-  - Os três eixos são paralelos e usam +X como eixo de rotação.
-  - As meshes são as STLs originais exportadas do Shapr3D.
-  - A garra e o Dynamixel 4 permanecem fora deste arquivo até o CAD da garra
-    e o frame final de montagem serem definidos.
-  Observação sobre o horn
-  O STL recebido do Dynamixel contém a carcaça e o horn como um único corpo.
-  No URDF, o centro do horn é a origem cinemática da junta. Visualmente, o
-  horn permanece junto com o corpo do motor porque não existe uma mesh separada
-  para ele; isso não altera a cinemática do braço.
+  Modelo canônico único do manipulador RAV.
+  Uso:
+  - dry-run: standalone:=true hardware_mode:=dry_run
+  - real:    standalone:=true hardware_mode:=real
+  - inclusão em outro Xacro: standalone permanece false
+  O Dynamixel 4 aciona um pinhão (gripper_pinion_joint, revoluto) que
+  engrena em duas cremalheiras (left_finger_joint/right_finger_joint,
+  prismáticas, mimic do pinhão). Isso é modelado e comandado em todos
+  os modos, inclusive real (Dynamixel ID 4, calibrado no wizard).
 -->
 <robot name="rav_manipulator" xmlns:xacro="http://www.ros.org/wiki/xacro">
-  <!--
-    Propriedades físicas provisórias para Gazebo.
-    Não interferem no controle dos Dynamixel reais.
-    Substituir futuramente por massas e tensores medidos/calculados.
-  -->
+  <xacro:arg name="standalone" default="false"/>
+  <xacro:arg name="hardware_mode" default="dry_run"/>
+  <xacro:property name="standalone_mode" value="$(arg standalone)"/>
+  <xacro:property name="selected_hardware_mode" value="$(arg hardware_mode)"/>
   <xacro:macro
       name="rav_provisional_inertial"
@@ -32,24 +28,93 @@
     </inertial>
   </xacro:macro>
-  <xacro:macro name="rav_manipulator"
-               params="parent_link mount_xyz:='0 0 0' mount_rpy:='0 0 0' use_fake_hardware:=false">
-    <!--
-      Referência geométrica extraída da pose CAD recebida, em metros.
-      J1 = eixo do horn do Dynamixel 1
-      J2 = eixo do horn do Dynamixel 2
-      J3 = eixo do horn do Dynamixel 3
-      As transforms J1→J2 e J2→J3 definem a pose zero no CAD. Não são os
-      comprimentos nominais do TCC; são as distâncias centro-a-centro reais
-      da montagem exportada.
-    -->
+  <xacro:macro
+      name="rav_manipulator"
+      params="parent_link
+              mount_xyz:='0 0 0'
+              mount_rpy:='0 0 0'
+              use_fake_hardware:=false
+              hardware_mode:='none'">
+    <!-- Geometria validada dos eixos do braço. -->
     <xacro:property name="j1_to_j2_y" value="0.000029639983"/>
     <xacro:property name="j1_to_j2_z" value="0.289118072919"/>
     <xacro:property name="j2_to_j3_y" value="-0.334030187591"/>
     <xacro:property name="j2_to_j3_z" value="-0.000015558969"/>
-    <!-- Limites provisórios: somente para RViz/MoveIt sem hardware real. -->
     <xacro:property name="joint_lower_limit" value="${-pi / 2.0}"/>
     <xacro:property name="joint_upper_limit" value="${ pi / 2.0}"/>
     <xacro:property name="joint_effort_limit" value="10.0"/>
     <xacro:property name="joint_velocity_limit" value="0.50"/>
+    <!--
+      Gripper: pinhão + cremalheira dupla, acionado pelo Dynamixel 4
+      (XM540-W270-R, encoder de 4096 ticks/volta).
+      Calibração validada no Dynamixel Wizard: motor centrado (tick
+      absoluto 2048 = 180°) é a posição fechada; abertura máxima segura
+      medida em tick absoluto 395 (34,72°). O delta real é 2048-395 =
+      1653 ticks (145,28°) — não 395, que é só a leitura absoluta do
+      lado aberto. gripper_max_travel foi originalmente calculado com
+      395 como se fosse o delta relativo; escalado proporcionalmente
+      por 1653/395 pra manter o raio do pinhão fisicamente plausível
+      (~7mm, compatível com o diâmetro visível da engrenagem na mesh).
+      O raio primitivo do pinhão é derivado dessa calibração e usado
+      como multiplicador nas juntas mimic dos dedos — para cremalheira
+      e pinhão, curso linear = raio x ângulo do pinhão é uma relação
+      exata, não uma aproximação.
+      Effort/velocity do pinhão vêm do torque de stall e da
+      velocidade sem carga do XM540-W270-R, interpolados para 12,7V
+      (ficha Robotis). Effort/velocity dos dedos são derivados do
+      pinhão pelo mesmo raio.
+    -->
+    <xacro:property name="gripper_max_travel_ticks" value="1653"/>
+    <xacro:property name="dxl_ticks_per_rev" value="4096"/>
+    <xacro:property name="gripper_max_travel" value="0.017749692"/>
+    <xacro:property
+        name="gripper_pinion_max_angle"
+        value="${gripper_max_travel_ticks * 2.0 * pi / dxl_ticks_per_rev}"/>
+    <xacro:property
+        name="gripper_pinion_radius"
+        value="${gripper_max_travel / gripper_pinion_max_angle}"/>
+    <xacro:property name="gripper_pinion_effort_limit" value="11.175"/>
+    <xacro:property name="gripper_pinion_velocity_limit" value="0.50"/>
+    <xacro:property
+        name="gripper_finger_effort_limit"
+        value="${gripper_pinion_effort_limit / gripper_pinion_radius}"/>
+    <xacro:property
+        name="gripper_finger_velocity_limit"
+        value="${gripper_pinion_velocity_limit * gripper_pinion_radius}"/>
+    <!--
+      dedo_esquerdo.stl/dedo_direito.stl foram exportados numa pose
+      aberta do CAD, não na posição fechada. gripper_max_travel (do
+      wizard, motor centrado = fechado) só cobre o curso fino de
+      abertura segura; sozinho ele não aproxima as pontas o
+      suficiente para tocarem em pinion=0.
+      gripper_finger_closed_offset é o deslocamento estático adicional
+      (por dedo) pra compensar isso. Base: vértice mais extremo (ápice)
+      de cada ponta nas meshes, resolvendo o deslocamento simétrico que
+      zera o vão entre elas (24,2159mm) — mas isso exagerou o fechamento
+      (dedos entrando um no outro). Corrigido com calibração visual: o
+      usuário comparou contra a gripper real e confirmou que
+      gripper_pinion_joint=20° no modelo antigo batia com o fechamento
+      real, então subtraímos o curso linear equivalente a 20° do
+      pinhão (raio x 20°) do valor bruto da mesh.
+    -->
+    <xacro:property name="gripper_finger_closed_offset_mesh_estimate" value="0.024215855"/>
+    <xacro:property name="gripper_finger_closed_offset_visual_correction_deg" value="20.0"/>
+    <xacro:property
+        name="gripper_finger_closed_offset"
+        value="${gripper_finger_closed_offset_mesh_estimate - gripper_pinion_radius * gripper_finger_closed_offset_visual_correction_deg * pi / 180.0}"/>
+    <!-- Origem CAD usada pelas meshes do punho e da gripper. -->
+    <xacro:property name="gripper_cad_origin_y" value="0.390472110866"/>
+    <xacro:property name="gripper_cad_origin_z" value="-1.011787152338"/>
+    <xacro:property
+        name="gripper_cad_origin"
+        value="0 ${gripper_cad_origin_y} ${gripper_cad_origin_z}"/>
+    <!--
+      Centro geométrico do pinhão (bounding box de pinhao.stl, dados
+      brutos da mesh), usado como origem da junta revoluta pra ela
+      girar no próprio eixo em vez de descrever um arco em torno da
+      origem de gripper_base_link.
+    -->
+    <xacro:property name="gripper_pinion_mesh_center_x" value="0.015923602"/>
+    <xacro:property name="gripper_pinion_mesh_center_y" value="-0.481112213"/>
+    <xacro:property name="gripper_pinion_mesh_center_z" value="1.013871002"/>
     <material name="rav_manipulator_motor">
       <color rgba="0.16 0.16 0.16 1.0"/>
@@ -58,9 +123,14 @@
       <color rgba="0.58 0.58 0.60 1.0"/>
     </material>
-    <!--
-      Mount externo. No modo standalone, o parent é manipulator_world.
-      Na integração final com o RAV, o parent será um frame da estrutura
-      interna e mount_xyz/mount_rpy serão medidos no CAD completo.
-    -->
+    <material name="rav_gripper_base_material">
+      <color rgba="0.20 0.20 0.22 1.0"/>
+    </material>
+    <material name="rav_gripper_finger_material">
+      <color rgba="0.58 0.58 0.60 1.0"/>
+    </material>
+    <material name="rav_gripper_pinion_material">
+      <color rgba="0.35 0.35 0.37 1.0"/>
+    </material>
+    <!-- Mount externo. -->
     <joint name="rav_manipulator_mount_joint" type="fixed">
       <parent link="${parent_link}"/>
@@ -68,8 +138,5 @@
       <origin xyz="${mount_xyz}" rpy="${mount_rpy}"/>
     </joint>
-    <!--
-      Dynamixel 1: a carcaça é fixada diretamente à estrutura interna do RAV.
-      O origin abaixo leva o centro do horn do STL para a origem do link.
-    -->
+    <!-- Dynamixel 1. -->
     <link name="manipulator_base_link">
       <xacro:rav_provisional_inertial
@@ -80,6 +147,7 @@
         <origin xyz="0 0.047471563258 -0.733684638388" rpy="0 0 0"/>
         <geometry>
-          <mesh filename="package://rav_description/meshes/manipulator/dynamixel_xm540.stl"
-                scale="0.001 0.001 0.001"/>
+          <mesh
+              filename="package://rav_description/meshes/manipulator/dynamixel_xm540.stl"
+              scale="0.001 0.001 0.001"/>
         </geometry>
         <material name="rav_manipulator_motor"/>
@@ -88,10 +156,10 @@
         <origin xyz="0 0.047471563258 -0.733684638388" rpy="0 0 0"/>
         <geometry>
-          <mesh filename="package://rav_description/meshes/manipulator/dynamixel_xm540.stl"
-                scale="0.001 0.001 0.001"/>
-        </geometry>
-      </collision>
-    </link>
-    <!-- J1: o horn do Dynamixel 1 movimenta U aço 1 + Link 1. -->
+          <mesh
+              filename="package://rav_description/meshes/manipulator/dynamixel_xm540.stl"
+              scale="0.001 0.001 0.001"/>
+        </geometry>
+      </collision>
+    </link>
     <joint name="shoulder_joint" type="revolute">
       <parent link="manipulator_base_link"/>
@@ -99,11 +167,11 @@
       <origin xyz="0 0 0" rpy="0 0 0"/>
       <axis xyz="1 0 0"/>
-      <limit lower="${joint_lower_limit}" upper="${joint_upper_limit}"
-             effort="${joint_effort_limit}" velocity="${joint_velocity_limit}"/>
-    </joint>
-    <!--
-      Conjunto rígido do primeiro elo:
-      U aço 1 + Link 1 + carcaça fixa do Dynamixel 2.
-    -->
+      <limit
+          lower="${joint_lower_limit}"
+          upper="${joint_upper_limit}"
+          effort="${joint_effort_limit}"
+          velocity="${joint_velocity_limit}"/>
+    </joint>
+    <!-- Link 1 e Dynamixel 2. -->
     <link name="shoulder_link">
       <xacro:rav_provisional_inertial
@@ -114,6 +182,7 @@
         <origin xyz="0 0.047471563258 -0.733684638388" rpy="0 0 0"/>
         <geometry>
-          <mesh filename="package://rav_description/meshes/manipulator/link_1_assembly.stl"
-                scale="0.001 0.001 0.001"/>
+          <mesh
+              filename="package://rav_description/meshes/manipulator/link_1_assembly.stl"
+              scale="0.001 0.001 0.001"/>
         </geometry>
         <material name="rav_manipulator_structure"/>
@@ -122,14 +191,15 @@
         <origin xyz="0 0.047471563258 -0.733684638388" rpy="0 0 0"/>
         <geometry>
-          <mesh filename="package://rav_description/meshes/manipulator/link_1_assembly.stl"
-                scale="0.001 0.001 0.001"/>
-        </geometry>
-      </collision>
-      <!-- Corpo do Dynamixel 2, fixo no Link 1. -->
+          <mesh
+              filename="package://rav_description/meshes/manipulator/link_1_assembly.stl"
+              scale="0.001 0.001 0.001"/>
+        </geometry>
+      </collision>
       <visual>
         <origin xyz="0 0.047501203241 -0.444566565469" rpy="0 0 0"/>
         <geometry>
-          <mesh filename="package://rav_description/meshes/manipulator/dynamixel_xm540.stl"
-                scale="0.001 0.001 0.001"/>
+          <mesh
+              filename="package://rav_description/meshes/manipulator/dynamixel_xm540.stl"
+              scale="0.001 0.001 0.001"/>
         </geometry>
         <material name="rav_manipulator_motor"/>
@@ -138,10 +208,10 @@
         <origin xyz="0 0.047501203241 -0.444566565469" rpy="0 0 0"/>
         <geometry>
-          <mesh filename="package://rav_description/meshes/manipulator/dynamixel_xm540.stl"
-                scale="0.001 0.001 0.001"/>
-        </geometry>
-      </collision>
-    </link>
-    <!-- J2: o horn do Dynamixel 2 movimenta U aço 2 + Link 2. -->
+          <mesh
+              filename="package://rav_description/meshes/manipulator/dynamixel_xm540.stl"
+              scale="0.001 0.001 0.001"/>
+        </geometry>
+      </collision>
+    </link>
     <joint name="elbow_joint" type="revolute">
       <parent link="shoulder_link"/>
@@ -149,11 +219,11 @@
       <origin xyz="0 ${j1_to_j2_y} ${j1_to_j2_z}" rpy="0 0 0"/>
       <axis xyz="1 0 0"/>
-      <limit lower="${joint_lower_limit}" upper="${joint_upper_limit}"
-             effort="${joint_effort_limit}" velocity="${joint_velocity_limit}"/>
-    </joint>
-    <!--
-      Conjunto rígido do segundo elo:
-      U aço 2 + Link 2 + carcaça fixa do Dynamixel 3.
-    -->
+      <limit
+          lower="${joint_lower_limit}"
+          upper="${joint_upper_limit}"
+          effort="${joint_effort_limit}"
+          velocity="${joint_velocity_limit}"/>
+    </joint>
+    <!-- Link 2 e Dynamixel 3. -->
     <link name="elbow_link">
       <xacro:rav_provisional_inertial
@@ -164,6 +234,7 @@
         <origin xyz="0 0.047441923275 -1.011802711307" rpy="0 0 0"/>
         <geometry>
-          <mesh filename="package://rav_description/meshes/manipulator/link_2_assembly.stl"
-                scale="0.001 0.001 0.001"/>
+          <mesh
+              filename="package://rav_description/meshes/manipulator/link_2_assembly.stl"
+              scale="0.001 0.001 0.001"/>
         </geometry>
         <material name="rav_manipulator_structure"/>
@@ -172,31 +243,31 @@
         <origin xyz="0 0.047441923275 -1.011802711307" rpy="0 0 0"/>
         <geometry>
-          <mesh filename="package://rav_description/meshes/manipulator/link_2_assembly.stl"
-                scale="0.001 0.001 0.001"/>
-        </geometry>
-      </collision>
-      <!--
-        Corpo do Dynamixel 3, fixo no Link 2.
-        O mesmo STL do Dynamixel 1 é reutilizado, mas com rotação de +90°
-        no eixo X. Assim, a carcaça fica alojada no interior da ponta do
-        Link 2, mantendo o centro do horn exatamente em J3.
-      -->
-      <visual>
-        <origin xyz="0 0.399654450797 0.047456004289" rpy="1.57079632679 0 0"/>
-        <geometry>
-          <mesh filename="package://rav_description/meshes/manipulator/dynamixel_xm540.stl"
-                scale="0.001 0.001 0.001"/>
+          <mesh
+              filename="package://rav_description/meshes/manipulator/link_2_assembly.stl"
+              scale="0.001 0.001 0.001"/>
+        </geometry>
+      </collision>
+      <visual>
+        <origin
+            xyz="0 0.399654450797 0.047456004289"
+            rpy="1.57079632679 0 0"/>
+        <geometry>
+          <mesh
+              filename="package://rav_description/meshes/manipulator/dynamixel_xm540.stl"
+              scale="0.001 0.001 0.001"/>
         </geometry>
         <material name="rav_manipulator_motor"/>
       </visual>
       <collision>
-        <origin xyz="0 0.399654450797 0.047456004289" rpy="1.57079632679 0 0"/>
-        <geometry>
-          <mesh filename="package://rav_description/meshes/manipulator/dynamixel_xm540.stl"
-                scale="0.001 0.001 0.001"/>
-        </geometry>
-      </collision>
-    </link>
-    <!-- J3: o horn do Dynamixel 3 movimenta U aço 3 e a futura garra. -->
+        <origin
+            xyz="0 0.399654450797 0.047456004289"
+            rpy="1.57079632679 0 0"/>
+        <geometry>
+          <mesh
+              filename="package://rav_description/meshes/manipulator/dynamixel_xm540.stl"
+              scale="0.001 0.001 0.001"/>
+        </geometry>
+      </collision>
+    </link>
     <joint name="wrist_joint" type="revolute">
       <parent link="elbow_link"/>
@@ -204,8 +275,11 @@
       <origin xyz="0 ${j2_to_j3_y} ${j2_to_j3_z}" rpy="0 0 0"/>
       <axis xyz="1 0 0"/>
-      <limit lower="${joint_lower_limit}" upper="${joint_upper_limit}"
-             effort="${joint_effort_limit}" velocity="${joint_velocity_limit}"/>
-    </joint>
-    <!-- U aço 3, onde o Dynamixel 4 será fixado quando a garra entrar. -->
+      <limit
+          lower="${joint_lower_limit}"
+          upper="${joint_upper_limit}"
+          effort="${joint_effort_limit}"
+          velocity="${joint_velocity_limit}"/>
+    </joint>
+    <!-- Punho e Dynamixel 4 visual. -->
     <link name="wrist_link">
       <xacro:rav_provisional_inertial
@@ -216,6 +290,7 @@
         <origin xyz="0 0.390472110866 -1.011787152338" rpy="0 0 0"/>
         <geometry>
-          <mesh filename="package://rav_description/meshes/manipulator/wrist_assembly.stl"
-                scale="0.001 0.001 0.001"/>
+          <mesh
+              filename="package://rav_description/meshes/manipulator/wrist_assembly.stl"
+              scale="0.001 0.001 0.001"/>
         </geometry>
         <material name="rav_manipulator_structure"/>
@@ -224,64 +299,193 @@
         <origin xyz="0 0.390472110866 -1.011787152338" rpy="0 0 0"/>
         <geometry>
-          <mesh filename="package://rav_description/meshes/manipulator/wrist_assembly.stl"
-                scale="0.001 0.001 0.001"/>
-        </geometry>
-      </collision>
-      <!--
-        Dynamixel 4: mesma geometria do XM540, rigidamente preso ao U aço 3.
-        Não é uma junta do braço: neste estágio ele é apenas a visualização e
-        a colisão do atuador que será usado futuramente para a gripper.
-        Correção de orientação:
-        - a rotação anterior em X colocava o corpo do motor na vertical;
-        - a pose abaixo parte da orientação de montagem anterior e adiciona
-          +90° no eixo Z, como no CAD do Shapr3D;
-        - a translação mantém o centro do horn no mesmo ponto do U aço 3.
-      -->
-      <visual>
-        <origin xyz="-0.718 -0.0619 0.0499"
-                rpy="1.57079632679 0 1.57079632679"/>
-        <geometry>
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
Commit message: ajustando paramentos manip

File: robotics_ws/src/rav_description/urdf/rav_manipulator.urdf.xacro (robot description, xacro)
@@ -43,5 +43,5 @@
     <xacro:property name="joint_upper_limit" value="${ pi / 2.0}"/>
     <xacro:property name="joint_effort_limit" value="10.0"/>
-    <xacro:property name="joint_velocity_limit" value="0.50"/>
+    <xacro:property name="joint_velocity_limit" value="1.0"/>
     <!--
       Gripper: pinhão + cremalheira dupla, acionado pelo Dynamixel 4
@@ -74,5 +74,5 @@
         value="${gripper_max_travel / gripper_pinion_max_angle}"/>
     <xacro:property name="gripper_pinion_effort_limit" value="11.175"/>
-    <xacro:property name="gripper_pinion_velocity_limit" value="0.50"/>
+    <xacro:property name="gripper_pinion_velocity_limit" value="1.0"/>
     <xacro:property
         name="gripper_finger_effort_limit"
@@ -561,6 +561,6 @@
           <param name="device">/dev/serial/by-id/usb-CM-900_ROBOTIS_Virtual_COM_Port-if00</param>
           <param name="baud">1000000</param>
-          <param name="profile_velocity">35</param>
-          <param name="profile_acceleration">12</param>
+          <param name="profile_velocity">70</param>
+          <param name="profile_acceleration">24</param>
         </hardware>
         <joint name="shoulder_joint">

File: robotics_ws/src/rav_manipulator_moveit_config/config/rav_manipulator_dynamixel_real.urdf.xacro (robot description, xacro)
@@ -18,6 +18,6 @@
       <param name="device">/dev/serial/by-id/usb-CM-900_ROBOTIS_Virtual_COM_Port-if00</param>
       <param name="baud">1000000</param>
-      <param name="profile_velocity">35</param>
-      <param name="profile_acceleration">12</param>
+      <param name="profile_velocity">70</param>
+      <param name="profile_acceleration">24</param>
     </hardware>
     <joint name="shoulder_joint">
