Commit message: Corrige transformada camera->manipulador e ajustes de pick/velocidade
Achada a causa raiz das coordenadas de visao saindo erradas pro pick:
faltava rotacao no camera_mount_joint (URDF), so tinha translacao.
Calculada via geometria real (braco em cam_pose, rotacao acumulada
quase zero) em vez de compensada com constante no codigo.

Outras correcoes da mesma investigacao:
- realtime_3d_inference: TF usava a transformacao mais recente em vez
  do timestamp exato da foto (bug real com camera montada em link
  movel); cy da CameraInfo com override, parametro cy_override
- manipulator_node: move_to_pose so tentava 2 orientacoes fixas pro
  IK, agora varre 24 (a cada 15 graus); IK_TIMEOUT_S reduzido de 2.0
  para 0.3s pra compensar; mensagem de erro do pick corrigida
- joint_limits: teto real de velocidade/aceleracao por junta pro
  braco (0.3) e gripper (0.5), gripper nao conseguia abrir/fechar a 1.0
- vision_pick_bridge: log da deteccao/coordenada usada antes do pick
- rav_vision: threshold de confianca 0.25 -> 0.75; remove
  tests_require obsoleto do setup.py

Co-Authored-By: Claude Sonnet 5 <noreply@anthropic.com>
Claude-Session: https://claude.ai/code/session_01AjK6BcToAnox5pXymERMgj

File: robotics_ws/src/rav_description/urdf/rav_manipulator.urdf.xacro (robot description, xacro)
@@ -487,4 +487,30 @@
       <origin xyz="0 -0.140 0.002" rpy="0 0 0"/>
     </joint>
+    <!-- Camera Astra (DaBai DCW) montada na ponta da gripper: 55mm em y e
+         40mm em z em relacao ao gripper_tcp (medido por Nathan). "camera_link"
+         precisa bater com o frame raiz publicado pelo astra_camera_node
+         (camera_name + "_link", default "camera_link") pra fechar a arvore de
+         TF entre a camera e o manipulador, sem isso o realtime_3d_inference
+         nunca consegue transformar as deteccoes pra manipulator_world.
+         Validado em 2026-09-12 com tf2_echo manipulator_world camera_link
+         vs medida de regua, braco parado: bateu (y dentro do erro de
+         regua, z exato), geometria da TRANSLACAO do mount esta certa.
+         Rotacao calculada em 2026-09-13 (nao mais chute rpy=0 0 0):
+         com o braco em cam_pose (shoulder+elbow+wrist ~= 0.036 rad, ou
+         seja quase sem rotacao acumulada do braco em si), comparamos
+         3 deteccoes reais (regua + move_to_pose manual) contra o que
+         o pipeline publicava em manipulator_world e vimos que faltava
+         exatamente uma rotacao de x,y,z -> z,-x,-y (matriz com
+         determinante +1, entao rotacao fisica valida, nao reflexo).
+         Isso corresponde a rpy = -90 0 -90 graus, coincide com a
+         mesma conversao fisico->optico que o driver da camera ja usa
+         entre camera_link e camera_color_optical_frame (conferido via
+         tf2_echo camera_link camera_color_optical_frame). -->
+    <link name="camera_link"/>
+    <joint name="camera_mount_joint" type="fixed">
+      <parent link="gripper_tcp"/>
+      <child link="camera_link"/>
+      <origin xyz="0 0.055 0.040" rpy="${-pi/2} 0 ${-pi/2}"/>
+    </joint>
     <!-- GenericSystem preservado para usos que instanciem a macro dessa forma. -->
     <xacro:if value="${use_fake_hardware}">

Commit message: robotics_ws: visão 3D calibrada, alinhamento da base com o Temi e ajustes de pick
Visão (rav_vision):
- Profundidade do objeto = superfície mais próxima na bbox inteira: a
  depth registrada fica deslocada da RGB e a mediana do centro caía no
  fundo (0.42 m virava 0.80 m, x saía 2x maior).
- fx_override=454 (camera_info diz 358; medido com régua).
- TransformListener com thread própria e fila de imagem depth=1 (YOLO na
  CPU travava o /tf e acumulava frames de ~2.5 s).
- vision_pick_bridge: idade máxima da detecção 5 s; z_offset_m (0).

Modelo/braço:
- camera_mount_joint rpy 0 0 -pi/2: a rotação óptica era aplicada duas
  vezes (URDF + driver), trocando x e z em manipulator_world.
- manipulator_node: pick_z_offset_m=+0.05 no alvo da garra.
- SRDF: poses atualizadas; rviz_real.launch.py pra reabrir só o RViz.

rav_task:
- teste_alinhamento: alinha a base com o objeto usando o yaw absoluto do
  Temi (calibrar_yaw salva yaw_prateleira), compensa o erro de ângulo de
  chegada, gira por yaw absoluto, anda mantendo rumo e avança 15 cm no
  fim (odometria); braço sempre em home com a base em movimento.
- start_task: alinhamento por giro antes do pick (girar_base); câmera
  com tf_publish_rate=0 no start_devices.

Co-Authored-By: Claude Opus 5.5 <noreply@anthropic.com>

File: robotics_ws/src/rav_description/urdf/rav_manipulator.urdf.xacro (robot description, xacro)
@@ -506,10 +506,18 @@
          mesma conversao fisico->optico que o driver da camera ja usa
          entre camera_link e camera_color_optical_frame (conferido via
-         tf2_echo camera_link camera_color_optical_frame). -->
+         tf2_echo camera_link camera_color_optical_frame).
+         Corrigido em 2026-10-05: justamente por coincidir com a conversao
+         do driver, o -90 0 -90 aplicava a rotacao optica DUAS vezes
+         (aqui + camera_link->camera_color_optical_frame), trocando x e z:
+         mover o objeto de lado mudava z em manipulator_world e mover pra
+         cima/baixo mudava x. So a profundidade (-y) batia, e era o unico
+         eixo validado (a ponte trava x=0). camera_link segue a convencao
+         ROS (x pra frente, z pra cima), entao aqui vai so a montagem
+         fisica: camera em pe olhando pra -y do gripper_tcp = yaw -90. -->
     <link name="camera_link"/>
     <joint name="camera_mount_joint" type="fixed">
       <parent link="gripper_tcp"/>
       <child link="camera_link"/>
-      <origin xyz="0 0.055 0.040" rpy="${-pi/2} 0 ${-pi/2}"/>
+      <origin xyz="0 0.055 0.040" rpy="0 0 ${-pi/2}"/>
     </joint>
     <!-- GenericSystem preservado para usos que instanciem a macro dessa forma. -->
