Commit message: add pacote moveit com .urdf para criacao de poses home, open, closed, attack no moveit com setup assistant

File: robotics_ws/src/rav_arm_moveit_config/config/rav_arm.urdf (robot description, URDF)
Before this commit: robot rav_arm, 9 links, 8 joints
Links:
- link arm_gripper_link_1: geometry collision box size=0.02 0.02 0.07; visual box size=0.02 0.04 0.07
- link arm_gripper_link_2: geometry collision box size=0.02 0.02 0.07; visual box size=0.02 0.04 0.07
Joints:
- joint arm_gripper_joint_1: limit lower=0.01 upper=0.03 effort=100.0 velocity=1.0 -> lower=0.01 upper=0.05 effort=100.0 velocity=1.0
- joint arm_gripper_joint_2: limit lower=-0.03 upper=-0.01 effort=100.0 velocity=1.0 -> lower=-0.05 upper=-0.01 effort=100.0 velocity=1.0; mimic (none) -> joint=arm_gripper_joint_1 multiplier=-1.0 offset=0.0
- joint arm_joint_2: limit lower=0.0 upper=6.28318 effort=300.0 velocity=1.0 -> lower=-0.3 upper=1.9787 effort=300.0 velocity=1.0
- joint arm_joint_3: limit lower=0.0 upper=6.28318 effort=300.0 velocity=1.0 -> lower=0.0 upper=2.3952 effort=300.0 velocity=1.0
- joint arm_joint_4: limit lower=-3.14159 upper=3.14159 effort=300.0 velocity=1.0 -> lower=-1 upper=1.5 effort=300.0 velocity=1.0

File: robotics_ws/src/rav_description/urdf/arm.urdf.xacro (robot description, xacro)
@@ -138,6 +138,6 @@
       <parent link="${prefix}link_2"/>
       <child link="${prefix}link_3"/>
-      <axis xyz="1 0 0"/>
-      <limit lower="0.0" upper="${M_PI * 2}" effort="300.0" velocity="1.0"/>
+      <axis xyz="-1 0 0"/>
+      <limit lower="4.0615" upper="6.2831" effort="300.0" velocity="1.0"/>
     </joint>
     <link name="${prefix}link_3">
